Commit message: adds skid steer bot test

File: test/skidsteerbot.xacro (robot description, xacro)
@@ -4,5 +4,5 @@
 Robot model taken from http://wiki.ros.org/pr2_mechanism/Tutorials/SImple%20URDF-Controller%20Example
 -->
-  <xacro:include filename="$(find diff_drive_controller)/test/wheel.xacro"/>
+  <xacro:include filename="$(find diff_drive_controller)/test/deg_to_rad.xacro"/>
   <xacro:property name="PI" value="3.1415926535897931"/>
   <!-- Constants for robot dimensions -->
@@ -11,4 +11,5 @@
   <xacro:property name="thickness" value="0.086" /> <!-- Link 2 -->
   <xacro:property name="axel_offset" value="0.05" /> <!-- Space btw top of beam and the each joint -->
+  <xacro:property name="y_offset" value="0.35" /> <!-- Offset for the wheels on the same side -->
   <!-- Links: inertial,visual,collision -->
   <link name="base_link">
@@ -52,8 +53,20 @@
   <!-- Wheels -->
   <wheel name="wheel_0" parent="base" radius="${wheel_radius}" thickness="${thickness}">
+    <origin xyz="${width/2+axel_offset} ${y_offset} 0" rpy="${-90 * deg_to_rad} 0 0"/>
+  </wheel>
+  <wheel name="wheel_1" parent="base" radius="${wheel_radius}" thickness="${thickness}">
     <origin xyz="${width/2+axel_offset} 0 0" rpy="${-90 * deg_to_rad} 0 0"/>
   </wheel>
-  <wheel name="wheel_1" parent="base" radius="${wheel_radius}" thickness="${thickness}">
+  <wheel name="wheel_2" parent="base" radius="${wheel_radius}" thickness="${thickness}">
+    <origin xyz="${width/2+axel_offset} ${-y_offset} 0" rpy="${-90 * deg_to_rad} 0 0"/>
+  </wheel>
+  <wheel name="wheel_3" parent="base" radius="${wheel_radius}" thickness="${thickness}">
+    <origin xyz="${-width/2+axel_offset} ${y_offset} 0" rpy="${-90 * deg_to_rad} 0 0"/>
+  </wheel>
+  <wheel name="wheel_4" parent="base" radius="${wheel_radius}" thickness="${thickness}">
     <origin xyz="${-width/2+axel_offset} 0 0" rpy="${-90 * deg_to_rad} 0 0"/>
+  </wheel>
+  <wheel name="wheel_5" parent="base" radius="${wheel_radius}" thickness="${thickness}">
+    <origin xyz="${-width/2+axel_offset} ${-y_offset} 0" rpy="${-90 * deg_to_rad} 0 0"/>
   </wheel>
   <!-- Colour -->
