Commit message: Fix test xacros

File: test/diffbot.xacro (robot description, xacro)
@@ -5,5 +5,5 @@
 -->
   <xacro:include filename="$(find diff_drive_controller)/test/wheel.xacro"/>
-  <xacro:property name="PI" value="3.1415926535897931"/>
+  <xacro:property name="deg_to_rad" value="0.01745329251994329577"/>
   <!-- Constants for robot dimensions -->
   <xacro:property name="width" value="0.5" /> <!-- Square dimensions (widthxwidth) of beams -->

File: test/skidsteerbot.xacro (robot description, xacro)
@@ -4,6 +4,6 @@
 Robot model taken from http://wiki.ros.org/pr2_mechanism/Tutorials/SImple%20URDF-Controller%20Example
 -->
-  <xacro:include filename="$(find diff_drive_controller)/test/deg_to_rad.xacro"/>
-  <xacro:property name="PI" value="3.1415926535897931"/>
+  <xacro:include filename="$(find diff_drive_controller)/test/wheel.xacro"/>
+  <xacro:property name="deg_to_rad" value="0.01745329251994329577"/>
   <!-- Constants for robot dimensions -->
   <xacro:property name="width" value="0.5" /> <!-- Square dimensions (widthxwidth) of beams -->
